File: reverse engineering gas leak sensor.kicad_sch (KiCad schematic)
At the start: 44 parts, among them Q1 BCX53, Q2 BCX53, Q3 BCX56, Q4 L8050QLT1G, Q5 BCX56, U3 MQ-4B, U4 NCP163ASN180T1G, U5 MC34063AG, U6 FT839NX, U7 MQ-4B

Commit message: stm
Parts:
- removed C1, C18, C2, C24, C26, C35, C4, C5: C, symbol Device:C
- removed R15, R39, R4: R, symbol Device:R
- removed U3, U7: MQ-4B, Sensor:MQ-6, symbol Sensor_Gas:MQ-6
- removed U4: NCP163ASN180T1G, Package_TO_SOT_SMD:SOT-23-5, symbol Regulator_Linear:NCP163ASN180T1G
- added C17, C22, C23, C25, C28, C29, C3 (x2), C31: C, symbol Device:C
- added L1: L, symbol Device:L
- added R22, R25, R28: R, symbol Device:R
- added U10: STM8S003F3P, Package_SO:TSSOP-20_4.4x6.5mm_P0.65mm, symbol MCU_ST_STM8:STM8S003F3P
- added U3: lcs docy2, Package_TO_SOT_SMD:SOT-23-5, symbol Regulator_Linear:LP2985-1.8
- added U4: AM5333M, Photon:SOT-223-3_TabPin2, symbol Photon:U_AMS1117-3.3_SOT-223_XBLW
- added U8: MQ-4B, Sensor:MQ-6, symbol Sensor_Gas:MQ-6
- added U9: ESP-12F, symbol ESP8266:ESP-12F
- renumbered C3 to C18, D5 to D9, R3 to R19
Connections:
- net GND: now also C16.1, C18.2, C27.2, U5.4 (GND), C17.2, C23.2, R25.1, U10.7 (VSS), U3.2 (GND), U4.1 (GND)
- net +12V: now reaches R19.1, U5.7 (Ipk)
- net +12V: now also U5.8 (DC)
- net at R19.2: now also U5.6 (Vin)
- net at U5.5 (Vfb): now also R25.2, R28.1
- net at D9.1 (K): now also R28.2; no longer C18.2
- net at C27.1: now also U3.4 (NC)
- net +5V: no longer names the net of C18.1
- net +5V: now also C17.1, L1.2
- new net: C23.1, U10.8 (VCAP)
- new net: C22.1, U10.9 (VDD)
- new net: C3.2, U8.2 (VH+)
- new net: C29.1, C31.1, U8.3 (A2)
- new net: L1.1, U8.5 (VH-)
- new net: C3.1, U4.3 (VO)
- new net: C28.1, C3.2
- new net: C22.2, C28.2
- new net: R22.1, U3.1 (VIN)
- new net: C25.1, U3.5 (VOUT)
- new net: C29.2, C31.2, R22.2
- new net: C25.2, U4.2 (VI)
- new net +5VA: C3.1, U3.3 (EN)
- no-connect marks 3 -> 2
Other:
- moved on the sheet: C16, C18, D9

Commit message: fixed recovered
Parts:
- removed C25, C3: C, symbol Device:C
- removed Q1, Q2: BCX53, Package_TO_SOT_SMD:SOT-89-3, symbol Transistor_BJT:BCX53
- removed Q3, Q5: BCX56, Package_TO_SOT_SMD:SOT-89-3, symbol Transistor_BJT:BCX56
- removed Q4: L8050QLT1G, easyeda2kicad:SOT-23-3_L2.9-W1.3-P1.90-LS2.4-BR, symbol easyeda2kicad:L8050QLT1G
- removed R1: R, symbol Device:R
- added C109, C24, C34, C35: C, symbol Device:C
- added D5, D8: 1N4148W, Diode_SMD:D_SOD-123, symbol Diode:1N4148W
- added ESD1, ESD2: ESD9B5.0ST5G, Diode_SMD:D_SOD-923, symbol Diode:ESD9B5.0ST5G
- added J2: Conn_01x05_Pin, symbol Connector:Conn_01x05_Pin
- added LED4: Inolux_IN-PI554FCH, LED_SMD:LED_Inolux_IN-PI554FCH_PLCC4_5.0x5.0mm_P3.2mm, symbol LED:Inolux_IN-PI554FCH
- added Q1: PNP, symbol Simulation_SPICE:PNP
- added Q10, Q11, Q2, Q3, Q4, Q5, Q6: NPN, symbol Simulation_SPICE:NPN
- added Q6, Q7: BCX53, Package_TO_SOT_SMD:SOT-89-3, symbol Transistor_BJT:BCX53
- added R13, R16, R20, R21, R23, R24, R26, R33, R34, R37, R39, R42, R44, R54, R56, R57, R6: R, symbol Device:R
- added SW1: SW_SPDT, symbol Switch:SW_SPDT
- U3: value lcs docy2 -> LPS DOCY2
- renumbered C3 to C38
Connections:
- net +12V: now also R56.2
- net GND: now also C28.2, C38.2, R6.1, C109.2, C24.2, ESD1.2 (A2), ESD2.1 (A1), LED4.1 (VSS), Q1.3 (E), Q10.3 (E), Q11.3 (E), Q3.3 (E), R39.2; no longer C27.2
- net at U10.12 (PB4): now also R37.1
- net at U10.13 (PC3): now also C35.1
- net at U10.16 (PC6): now also R23.1, R54.1
- net at U10.17 (PC7): now also R55.2, Q5.2 (B), R24.1, R24.2
- net at U10.19 (PD2): now also R6.2
- net at U10.20 (PD3): now also R42.1
- net at U10.4 (NRST): now also R44.2
- net at U10.9 (VDD): now also C22.2; no longer C22.1
- net at R2.2: now also Q2.2 (B)
- net at D3.1 (K): now also D2.1 (K), D4.2 (A), Q1.1 (C), Q2.1 (C)
- net at U8.1 (A1): now also C29.1, C31.1, U8.3 (A2)
- net at U8.2 (VH+): now also C29.2, C31.2, U3.1 (VOUT)
- net at U8.4 (B2): now also U8.6 (B1), R39.1
- net at C38.1, U4.3 (VO): now also C28.1, U9.8 (VCC)
- net at R55.1: now also Q11.2 (B)
- net at D2.2 (A): no longer R6.1
- net at U3.4 (NC): now also C27.2, U3.5 (VIN); no longer C27.1
- net at R22.1: now also Q6.2 (C); no longer U3.1 (VIN)
- net +5V: now reaches U4.2 (VI)
- net +5V: now also C22.1, C27.1, C34.1, R44.1
- net +5VA: no longer names the net of U3.3 (EN)
- net +5VA: now also R33.1
- new net: Q6.1 (C), R13.1
- new net: R13.2, R56.1
- new net: D5.2 (A), ESD1.1 (A1), J2.1 (Pin_1)
- new net: C109.1, R57.2
- new net: R34.1, R37.2
- new net: LED4.4 (DO), R26.1
- new net: Q3.1 (C), Q4.1 (C)
- new net: Q11.1 (C), Q3.2 (B), R20.1
- new net: Q6.1 (B), R34.2
- new net: Q6.2 (B), R23.2
- new net: Q6.3 (E), R20.2
- new net: Q4.2 (B), R57.1
- new net: D5.1 (K), Q4.3 (E)
- new net: Q5.1 (C), R16.2
- new net: Q5.3 (E), R21.2
- new net: C34.2, R33.2
- new net: D8.2 (A), ESD2.2 (A2), J2.2 (Pin_2)
- new net: Q6.3 (E), Q7.3 (E)
- new net: LED4.2 (DIN), R22.2
- new net: Q10.2 (B), R54.2
- new net: C24.1, R42.2
- new net: Q1.2 (B), Q10.1 (C), R21.1
- no-connect marks 2 -> 4
Other:
- moved on the sheet: C102, C104, C109, C16, C17, C18, C22, C23, C27, C28, C29, C31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
