File: _autosave-reverse engineering gas leak sensor.kicad_sch (KiCad schematic)
At the start: 89 parts, among them J2 Conn_01x05_Pin, Q1 PNP, Q10 NPN, Q11 NPN, Q2 NPN, Q3 NPN, Q4 NPN, Q5 NPN, Q6 BCX53, Q6 NPN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

Commit message: thursday 15th
Parts:
- removed C35: C, symbol Device:C
- removed Q6, Q7: BCX53, Package_TO_SOT_SMD:SOT-89-3, symbol Transistor_BJT:BCX53
- added C26: C, symbol Device:C
- added Q7, Q8: PNP, symbol Simulation_SPICE:PNP
- added R31, R36, R45, R46, R9: R, symbol Device:R
- added U1: SC5180B, symbol RELibrary:SC5180B
- renumbered R22 to R10
Connections:
- net +5V: now also R35.1, U10.9 (VDD), U3.4 (NC), U3.5 (VIN), Q8.3 (E), R36.1; no longer R44.2
- net GND: now also C22.2, C27.2, U3.2 (GND), U4.1 (GND), C26.2, R45.1; no longer LED4.1 (VSS)
- net at U10.13 (PC3): now also R35.2
- net tp1: now reaches U10.10 (PA3)
- net at U10.11 (PB5): now also R31.2
- net SC5180B_PIN2: now reaches U10.6 (PA2)
- net at C29.1, C31.1, U8.1 (A1)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: now also R46.2
- net at R34.1, R37.2: now also Q7.2 (B)
- net at LED4.4 (DO): no longer R26.1
- net at R26.2: now also Q8.1 (C), R9.2
- net at R34.2: now also Q7.3 (E)
- net at R10.1: now also Q7.1 (C)
- net at LED4.2 (DIN): no longer R10.2
- net at U9.3 (GPIO_0): no longer R35.2
- new net: Q8.2 (B), R31.1, R36.2
- new net 5-33_VoltRegulatorIn: R44.2
- new net LED2: R10.2, R9.1
- new net LED4: R26.1
- new net STM_PIN14: C26.1, R45.2, R46.1
Other:
- moved on the sheet: C27, C34, LED4, R33, R34
