File: esp connections.kicad_sch (KiCad schematic)
At the start: 3 parts, among them U1 ESP-12F, U2 STM8S003F3P

Commit message: stm
Other:
- moved on the sheet: D1, U1
Changed lines of the file:
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@@
 	(wire
 		(pts
-			(xy 88.9 114.3) (xy 69.85 114.3)
-		)
-		(stroke
-			(width 0)
-			(type default)
-		)
-	)
-	(wire
-		(pts
-			(xy 69.85 114.3) (xy 69.85 77.47)
-		)
-		(stroke
-			(width 0)
-			(type default)
-		)
-	)
-	(wire
-		(pts
-			(xy 134.62 114.3) (xy 134.62 118.11)
-		)
-		(stroke
-			(width 0)
-			(type default)
-		)
-	)
-	(wire
-		(pts
-			(xy 148.59 109.22) (xy 148.59 83.82)
-		)
-		(stroke
-			(width 0)
-			(type default)
-		)
-	)
-	(wire
-		(pts
-			(xy 134.62 109.22) (xy 148.59 109.22)
+			(xy 39.37 58.42) (xy 20.32 58.42)
+		)
+		(stroke
+			(width 0)
+			(type default)
+		)
+	)
+	(wire
+		(pts
+			(xy 20.32 58.42) (xy 20.32 21.59)
+		)
+		(stroke
+			(width 0)
+			(type default)
+		)
+	)
+	(wire
+		(pts
+			(xy 85.09 58.42) (xy 85.09 62.23)
+		)
+		(stroke
+			(width 0)
+			(type default)
+		)
+	)
+	(wire
+		(pts
+			(xy 99.06 53.34) (xy 99.06 27.94)
+		)
+		(stroke
+			(width 0)
+			(type default)
+		)
+	)
+	(wire
+		(pts
+			(xy 85.09 53.34) (xy 99.06 53.34)
 		)
 		(stroke
@@
 	(symbol
 		(lib_id "power:GND")
-		(at 134.62 118.11 0)
+		(at 85.09 62.23 0)
 		(unit 1)
 		(exclude_from_sim no)
@@
 		(fields_autoplaced yes)
 		(property "Reference" "#PWR01"
-			(at 134.62 124.46 0)
+			(at 85.09 68.58 0)
 			(effects
 				(font
@@
 		)
 		(property "Value" "GND"
-			(at 134.62 123.19 0)
+			(at 85.09 67.31 0)
 			(effects
 				(font
@@
 		)
 		(property "Footprint" ""
-			(at 134.62 118.11 0)
+			(at 85.09 62.23 0)
 			(effects
 				(font
@@
 		)
 		(property "Datasheet" ""
-			(at 134.62 118.11 0)
+			(at 85.09 62.23 0)
 			(effects
 				(font
@@
 		)
 		(property "Description" "Power symbol creates a global label with name \"GND\" , ground"
-			(at 134.62 118.11 0)
+			(at 85.09 62.23 0)
 			(effects
 				(font
@@
 	(symbol
 		(lib_id "ESP8266:ESP-12F")
-		(at 111.76 104.14 0)
+		(at 62.23 48.26 0)
 		(unit 1)
 		(exclude_from_sim no)
@@
 		(fields_autoplaced yes)
 		(property "Reference" "U1"
-			(at 111.76 83.82 0)
+			(at 62.23 27.94 0)
 			(effects
 				(font
@@
 		)
 		(property "Value" "ESP-12F"
-			(at 111.76 86.36 0)
+			(at 62.23 30.48 0)
 			(effects
 				(font
@@
 		)
 		(property "Footprint" ""
-			(at 111.76 104.14 0)
+			(at 62.23 48.26 0)
 			(effects
 				(font
@@
 		)
 		(property "Datasheet" "http://l0l.org.uk/2014/12/esp8266-modules-hardware-guide-gotta-catch-em-all/"
-			(at 111.76 104.14 0)
+			(at 62.23 48.26 0)
 			(effects
 				(font
@@
 		)
 		(property "Description" "ESP8266 ESP-12E module, 22 pins, 2mm, PCB antenna"
-			(at 111.76 104.14 0)
+			(at 62.23 48.26 0)
 			(effects
 				(font
@@
 	(symbol
 		(lib_id "Device:LED_ABGR")
-		(at 148.59 78.74 90)
+		(at 99.06 22.86 90)
 		(unit 1)
 		(exclude_from_sim no)
@@
 		(fields_autoplaced yes)
 		(property "Reference" "D1"
-			(at 157.48 77.4699 90)
+			(at 107.95 21.5899 90)
 			(effects
 				(font
@@
 		)
 		(property "Value" "LED_ABGR"
-			(at 157.48 80.0099 90)
+			(at 107.95 24.1299 90)
 			(effects
 				(font
@@
 		)
 		(property "Footprint" ""
-			(at 149.86 78.74 0)
+			(at 100.33 22.86 0)
 			(effects
 				(font
@@
 		)
 		(property "Datasheet" "~"
-			(at 149.86 78.74 0)
+			(at 100.33 22.86 0)
 			(effects
 				(font
@@
 		)
 		(property "Description" "RGB LED, anode/blue/green/red"
-			(at 148.59 78.74 0)
+			(at 99.06 22.86 0)
 			(effects
 				(font
@@
 	(symbol
 		(lib_id "power:VCC")
-		(at 69.85 77.47 0)
+		(at 20.32 21.59 0)
 		(unit 1)
 		(exclude_from_sim no)
@@
 		(fields_autoplaced yes)
 		(property "Reference" "#PWR02"
-			(at 69.85 81.28 0)
+			(at 20.32 25.4 0)
 			(effects
 				(font
@@
 		)
 		(property "Value" "VCC +3.3v"
-			(at 69.85 72.39 0)
+			(at 20.32 16.51 0)
 			(effects
 				(font
@@
 		)
 		(property "Footprint" ""
-			(at 69.85 77.47 0)
+			(at 20.32 21.59 0)
 			(effects
 				(font
@@
 		)
 		(property "Datasheet" ""
-			(at 69.85 77.47 0)
+			(at 20.32 21.59 0)
 			(effects
 				(font
@@
 		)
 		(property "Description" "Power symbol creates a global label with name \"VCC\""
-			(at 69.85 77.47 0)
-			(effects
-				(font
+			(at 20.32 21.59 0)
+			(effects
+				(font

Commit message: thursday 15th
Parts:
- removed D1: LED_ABGR, symbol Device:LED_ABGR
- removed U1: ESP-12F, symbol ESP8266:ESP-12F
- removed U2: STM8S003F3P, Package_SO:TSSOP-20_4.4x6.5mm_P0.65mm, symbol MCU_ST_STM8:STM8S003F3P
- added C22, C4, C6, C7, C8: C, symbol Device:C
- added LED1: Inolux_IN-PI554FCH, LED_SMD:LED_Inolux_IN-PI554FCH_PLCC4_5.0x5.0mm_P3.2mm, symbol LED:Inolux_IN-PI554FCH
- added Q12, Q13, Q8, Q9: NPN, symbol Simulation_SPICE:NPN
- added Q14, Q15: BCX53, Package_TO_SOT_SMD:SOT-89-3, symbol Transistor_BJT:BCX53
- added R1, R10, R11, R12, R14, R15, R17, R18, R27, R29, R3, R30, R31, R4, R5, R7, R8, R9: R, symbol Device:R
- added SW2: SW_SPDT, symbol Switch:SW_SPDT
- added U7: STM8S003F3P, Package_SO:TSSOP-20_4.4x6.5mm_P0.65mm, symbol MCU_ST_STM8:STM8S003F3P
Connections:
- net GND: now also C4.2, LED1.1 (VSS), Q8.3 (E), Q9.3 (E), U7.7 (VSS)
- new net: C4.1, U7.8 (VCAP)
- new net: R18.1, U7.1 (PD4)
- new net: C7.2, R18.2
- new net: R30.2, U7.19 (PD2)
- new net: R10.2, R11.1
- new net: LED1.4 (DO), R27.1
- new net: R15.1, U7.2 (PD5)
- new net: R14.1, U7.12 (PB4)
- new net: R14.2, R17.1
- new net: C6.1, U7.13 (PC3)
- new net: R3.1, R8.1, U7.16 (PC6)
- new net: Q13.2 (B), R12.1, R12.2, R7.2, U7.17 (PC7)
- new net: R31.1, U7.20 (PD3)
- new net: R9.2, U7.4 (NRST)
- new net: C22.2, U7.9 (VDD)
- new net: Q8.2 (B), R3.2
- new net: Q13.1 (C), R5.2
- new net: Q12.1 (C), R10.1
- new net: Q12.2 (B), R8.2
- new net: Q12.3 (E), R1.2
- new net: Q14.1 (B), R17.2
- new net: Q14.2 (C), R29.1
- new net: Q14.3 (E), Q15.3 (E)
- new net: Q9.2 (B), R7.1
- new net: Q9.1 (C), R1.1
- new net: Q13.3 (E), R4.2
- new net: C8.1, R31.2
- new net: LED1.2 (DIN), R29.2
- new net +12V: R11.2
- new net +3.3v: C22.1
- new net +5V: R9.1
- new net B1_Sensor: C8.2
- new net ProtectionQ1: Q8.1 (C), R4.1
- no-connect marks 0 -> 2

Commit message: new
Parts:
- removed C22, C4, C6, C7, C8: C, symbol Device:C
- removed LED1: Inolux_IN-PI554FCH, LED_SMD:LED_Inolux_IN-PI554FCH_PLCC4_5.0x5.0mm_P3.2mm, symbol LED:Inolux_IN-PI554FCH
- removed Q12, Q13, Q8, Q9: NPN, symbol Simulation_SPICE:NPN
- removed Q14, Q15: BCX53, Package_TO_SOT_SMD:SOT-89-3, symbol Transistor_BJT:BCX53
- removed R1, R10, R11, R12, R14, R15, R17, R18, R27, R29, R3, R30, R31, R4, R5, R7, R8, R9: R, symbol Device:R
- removed SW2: SW_SPDT, symbol Switch:SW_SPDT
- removed U7: STM8S003F3P, Package_SO:TSSOP-20_4.4x6.5mm_P0.65mm, symbol MCU_ST_STM8:STM8S003F3P
Connections:
- no-connect marks 2 -> 0
