File: new re gas leak schematic.kicad_sch (KiCad schematic)
At the start: 95 parts, among them J2 Conn_01x05_Pin, Q1 PNP, Q10 NPN, Q11 NPN, Q2 NPN, Q3 NPN, Q4 NPN, Q5 NPN, Q6 NPN, Q7 PNP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

Commit message: new
Parts:
- added C1: C, symbol Device:C
Connections:
- net STM_PIN14: now also U10.14 (PC4)
Other:
- moved on the sheet: C27
Changed lines of the file:
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@@
 	)
 	(junction
+		(at 200.66 80.01)
+		(diameter 0)
+		(color 0 0 0 0)
+	)
+	(junction
 		(at 62.23 67.31)
 		(diameter 0)
@@
 	)
 	(junction
-		(at 210.82 91.44)
-		(diameter 0)
-		(color 0 0 0 0)
-	)
-	(junction
 		(at 269.24 142.24)
 		(diameter 0)
@@
 	)
 	(junction
-		(at 250.19 120.65)
+		(at 208.28 91.44)
 		(diameter 0)
 		(color 0 0 0 0)
 	)
 	(junction
-		(at 36.83 199.39)
+		(at 250.19 120.65)
 		(diameter 0)
 		(color 0 0 0 0)
 	)
 	(junction
-		(at 67.31 219.71)
+		(at 36.83 199.39)
 		(diameter 0)
 		(color 0 0 0 0)
 	)
 	(junction
-		(at 210.82 80.01)
+		(at 67.31 219.71)
 		(diameter 0)
 		(color 0 0 0 0)
@@
 	(wire
 		(pts
-			(xy 190.5 91.44) (xy 210.82 91.44)
+			(xy 190.5 91.44) (xy 208.28 91.44)
 		)
 		(stroke
@@
 	(wire
 		(pts
-			(xy 200.66 82.55) (xy 208.28 82.55)
-		)
-		(stroke
-			(width 0)
-			(type default)
-		)
-	)
-	(wire
-		(pts
 			(xy 389.89 113.03) (xy 386.08 113.03)
 		)
@@
 	(wire
 		(pts
-			(xy 210.82 91.44) (xy 210.82 92.71)
+			(xy 208.28 91.44) (xy 208.28 92.71)
 		)
 		(stroke
@@
 	(wire
 		(pts
-			(xy 210.82 91.44) (xy 227.33 91.44)
+			(xy 208.28 91.44) (xy 227.33 91.44)
 		)
 		(stroke
@@
 	(wire
 		(pts
-			(xy 210.82 83.82) (xy 210.82 80.01)
+			(xy 208.28 83.82) (xy 208.28 80.01)
 		)
 		(stroke
@@
 	(wire
 		(pts
-			(xy 219.71 80.01) (xy 210.82 80.01)
-		)
-		(stroke
-			(width 0)
-			(type default)
-		)
-	)
-	(wire
-		(pts
 			(xy 59.69 36.83) (xy 63.5 36.83)
 		)
@@
 	(wire
 		(pts
-			(xy 208.28 82.55) (xy 208.28 80.01)
+			(xy 236.22 184.15) (xy 236.22 120.65)
 		)
 		(stroke
@@
 	(wire
 		(pts
-			(xy 236.22 184.15) (xy 236.22 120.65)
+			(xy 200.66 80.01) (xy 200.66 82.55)
 		)
 		(stroke
@@
 	(wire
 		(pts
-			(xy 210.82 80.01) (xy 208.28 80.01)
-		)
-		(stroke
-			(width 0)
-			(type default)
-		)
-	)
-	(wire
-		(pts
 			(xy 36.83 199.39) (xy 36.83 209.55)
 		)
@@
 	(wire
 		(pts
+			(xy 208.28 80.01) (xy 219.71 80.01)
+		)
+		(stroke
+			(width 0)
+			(type default)
+		)
+	)
+	(wire
+		(pts
 			(xy 90.17 227.33) (xy 90.17 228.6)
 		)
@@
 		)
 	)
+	(global_label "STM_PIN14"
+		(shape input)
+		(at 251.46 113.03 180)
+		(fields_autoplaced yes)
+		(effects
+			(font
+				(size 1.27 1.27)
+			)
+			(justify right)
+		)
+		(property "Intersheetrefs" "${INTERSHEET_REFS}"
+			(at 238.2544 113.03 0)
+			(effects
+				(font
+					(size 1.27 1.27)
+				)
+				(justify right)
+				(hide yes)
+			)
+		)
+	)
 	(global_label "SC5180B_PIN4"
 		(shape input)
@@
 	(symbol
 		(lib_id "power:GND")
-		(at 210.82 92.71 0)
+		(at 208.28 92.71 0)
 		(unit 1)
 		(exclude_from_sim no)
@@
 		(fields_autoplaced yes)
 		(property "Reference" "#PWR010"
-			(at 210.82 99.06 0)
+			(at 208.28 99.06 0)
 			(effects
 				(font
@@
 		)
 		(property "Value" "GND"
-			(at 210.82 97.79 0)
+			(at 208.28 97.79 0)
 			(effects
 				(font
@@
 		)
 		(property "Footprint" ""
-			(at 210.82 92.71 0)
+			(at 208.28 92.71 0)
 			(effects
 				(font
@@
 		)
 		(property "Datasheet" ""
-			(at 210.82 92.71 0)
+			(at 208.28 92.71 0)
 			(effects
 				(font
@@
 		)
 		(property "Description" "Power symbol creates a global label with name \"GND\" , ground"
-			(at 210.82 92.71 0)
+			(at 208.28 92.71 0)
 			(effects
 				(font
@@
 	(symbol
 		(lib_id "Device:C")
-		(at 210.82 87.63 0)
+		(at 208.28 87.63 0)
 		(unit 1)
 		(exclude_from_sim no)
@@
 		(dnp no)
 		(property "Reference" "C27"
-			(at 216.916 87.63 90)
+			(at 214.376 87.63 90)
 			(effects
 				(font
@@
 		)
 		(property "Value" "C"
-			(at 214.376 87.63 90)
+			(at 211.836 87.63 90)
 			(effects
 				(font
@@
 		)
 		(property "Footprint" ""
-			(at 211.7852 91.44 0)
+			(at 209.2452 91.44 0)
 			(effects
 				(font
@@
 		)
 		(property "Datasheet" "~"
-			(at 210.82 87.63 0)
+			(at 208.28 87.63 0)
 			(effects
 				(font
@@
 		)
 		(property "Description" "Unpolarized capacitor"
-			(at 210.82 87.63 0)
+			(at 208.28 87.63 0)
 			(effects
 				(font
@@
 					(unit 1)
 				)
+			)
+		)
+	)
+	(symbol
+		(lib_id "Device:C")
+		(at 257.81 166.37 0)
+		(unit 1)
+		(exclude_from_sim no)
+		(in_bom yes)
+		(on_board yes)
+		(dnp no)
+		(property "Reference" "C1"
+			(at 263.906 166.37 90)
+			(effects
+				(font
+					(size 1.27 1.27)
+				)
+			)
+		)
+		(property "Value" "C"
+			(at 261.366 166.37 90)
+			(effects
+				(font
+					(size 1.27 1.27)
+				)
+			)
+		)
+		(property "Footprint" ""
+			(at 258.7752 170.18 0)
+			(effects
+				(font
+					(size 1.27 1.27)
+				)
+				(hide yes)
+			)
+		)
+		(property "Datasheet" "~"
+			(at 257.81 166.37 0)
+			(effects
+				(font
+					(size 1.27 1.27)
+				)
+				(hide yes)
+			)
+		)
+		(property "Description" "Unpolarized capacitor"
+			(at 257.81 166.37 0)
+			(effects
+				(font
+					(size 1.27 1.27)
+				)
+				(hide yes)
+			)
+		)
+		(pin "2"
+		)
+		(pin "1"
+		)
+		(instances
+			(project "reverse engineering gas leak sensor"
+				(path "/408e2ccf-0846-4a9f-a9c5-211b02235e03"
+					(reference "C1")
+					(unit 1)
+				)
