File: BLOCK_DIAGRAM/block diagram/untitled.kicad_sch (KiCad schematic)
At the start: 15 parts, among them Q1 NMOS, U1 ESP32-C3-WROOM-02, U2 STM8S003F3P, U3 MQ-4M, U4 5-3v3, U5 12-5v, U6 220-12v

Commit message: edited the connections of the 220-5 (added the RLC) and added RLC for en pullup and 3v3 of esp
Parts:
- renumbered R3 to R1, R4 to R2, R2 to R3, R1 to R4, U6 to U1, U5 to U2, U4 to U3, U3 to U4, U2 to U5, U1 to U6
Changed lines of the file:
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@@
 		(dnp no)
 		(fields_autoplaced yes)
-		(property "Reference" "U6"
+		(property "Reference" "U1"
 			(at 44.0533 48.26 0)
 			(effects
@@
 		(instances
 			(project "block diagram"
-				(path "/290c0625-1e23-4ef7-8910-f1eb5378fd87/46229e74-cb6e-4f48-8e10-26ccf9ffc6c9"
-					(reference "U6")
+				(path "/290c0625-1e23-4ef7-8910-f1eb5378fd87/645251e2-b784-4e24-8757-44ff6e2afd31"
+					(reference "U1")
 					(unit 1)
 				)
@@
 		(dnp no)
 		(fields_autoplaced yes)
-		(property "Reference" "U5"
+		(property "Reference" "U2"
 			(at 71.9933 48.26 0)
 			(effects
@@
 		(instances
 			(project "block diagram"
-				(path "/290c0625-1e23-4ef7-8910-f1eb5378fd87/46229e74-cb6e-4f48-8e10-26ccf9ffc6c9"
-					(reference "U5")
+				(path "/290c0625-1e23-4ef7-8910-f1eb5378fd87/645251e2-b784-4e24-8757-44ff6e2afd31"
+					(reference "U2")
 					(unit 1)
 				)
@@
 		(dnp no)
 		(fields_autoplaced yes)
-		(property "Reference" "U3"
+		(property "Reference" "U4"
 			(at 136.7633 54.61 0)
 			(effects
@@
 		(instances
 			(project "block diagram"
-				(path "/290c0625-1e23-4ef7-8910-f1eb5378fd87/46229e74-cb6e-4f48-8e10-26ccf9ffc6c9"
-					(reference "U3")
+				(path "/290c0625-1e23-4ef7-8910-f1eb5378fd87/645251e2-b784-4e24-8757-44ff6e2afd31"
+					(reference "U4")
 					(unit 1)
 				)
@@
 		(instances
 			(project "block diagram"
-				(path "/290c0625-1e23-4ef7-8910-f1eb5378fd87/46229e74-cb6e-4f48-8e10-26ccf9ffc6c9"
+				(path "/290c0625-1e23-4ef7-8910-f1eb5378fd87/645251e2-b784-4e24-8757-44ff6e2afd31"
 					(reference "C1")
 					(unit 1)
@@
 		(instances
 			(project "block diagram"
-				(path "/290c0625-1e23-4ef7-8910-f1eb5378fd87/46229e74-cb6e-4f48-8e10-26ccf9ffc6c9"
+				(path "/290c0625-1e23-4ef7-8910-f1eb5378fd87/645251e2-b784-4e24-8757-44ff6e2afd31"
 					(reference "Q1")
 					(unit 1)
@@
 		(on_board yes)
 		(dnp no)
-		(property "Reference" "R1"
+		(property "Reference" "R4"
 			(at 209.55 48.26 0)
 			(effects
@@
 		(instances
 			(project "block diagram"
-				(path "/290c0625-1e23-4ef7-8910-f1eb5378fd87/46229e74-cb6e-4f48-8e10-26ccf9ffc6c9"
-					(reference "R1")
+				(path "/290c0625-1e23-4ef7-8910-f1eb5378fd87/645251e2-b784-4e24-8757-44ff6e2afd31"
+					(reference "R4")
 					(unit 1)
 				)
@@
 		(on_board yes)
 		(dnp no)
-		(property "Reference" "R2"
+		(property "Reference" "R3"
 			(at 165.1 40.64 0)
 			(effects
@@
 		(instances
 			(project "block diagram"
-				(path "/290c0625-1e23-4ef7-8910-f1eb5378fd87/46229e74-cb6e-4f48-8e10-26ccf9ffc6c9"
-					(reference "R2")
+				(path "/290c0625-1e23-4ef7-8910-f1eb5378fd87/645251e2-b784-4e24-8757-44ff6e2afd31"
+					(reference "R3")
 					(unit 1)
 				)
@@
 		(dnp no)
 		(fields_autoplaced yes)
-		(property "Reference" "U2"
+		(property "Reference" "U5"
 			(at 187.5633 35.56 0)
 			(effects
@@
 		(instances
 			(project "block diagram"
-				(path "/290c0625-1e23-4ef7-8910-f1eb5378fd87/46229e74-cb6e-4f48-8e10-26ccf9ffc6c9"
-					(reference "U2")
+				(path "/290c0625-1e23-4ef7-8910-f1eb5378fd87/645251e2-b784-4e24-8757-44ff6e2afd31"
+					(reference "U5")
 					(unit 1)
 				)
@@
 		(instances
 			(project "block diagram"
-				(path "/290c0625-1e23-4ef7-8910-f1eb5378fd87/46229e74-cb6e-4f48-8e10-26ccf9ffc6c9"
+				(path "/290c0625-1e23-4ef7-8910-f1eb5378fd87/645251e2-b784-4e24-8757-44ff6e2afd31"
 					(reference "R6")
 					(unit 1)
@@
 		(instances
 			(project "block diagram"
-				(path "/290c0625-1e23-4ef7-8910-f1eb5378fd87/46229e74-cb6e-4f48-8e10-26ccf9ffc6c9"
+				(path "/290c0625-1e23-4ef7-8910-f1eb5378fd87/645251e2-b784-4e24-8757-44ff6e2afd31"
 					(reference "#PWR01")
 					(unit 1)
@@
 		(dnp no)
 		(fields_autoplaced yes)
-		(property "Reference" "U1"
+		(property "Reference" "U6"
 			(at 237.0933 36.83 0)
 			(effects
@@
 		(instances
 			(project "block diagram"
-				(path "/290c0625-1e23-4ef7-8910-f1eb5378fd87/46229e74-cb6e-4f48-8e10-26ccf9ffc6c9"
-					(reference "U1")
+				(path "/290c0625-1e23-4ef7-8910-f1eb5378fd87/645251e2-b784-4e24-8757-44ff6e2afd31"
+					(reference "U6")
 					(unit 1)
 				)
@@
 		(on_board yes)
 		(dnp no)
-		(property "Reference" "R4"
+		(property "Reference" "R2"
 			(at 161.29 45.72 0)
 			(effects
@@
 		(instances
 			(project "block diagram"
-				(path "/290c0625-1e23-4ef7-8910-f1eb5378fd87/46229e74-cb6e-4f48-8e10-26ccf9ffc6c9"
-					(reference "R4")
+				(path "/290c0625-1e23-4ef7-8910-f1eb5378fd87/645251e2-b784-4e24-8757-44ff6e2afd31"
+					(reference "R2")
 					(unit 1)
 				)
@@
 		(instances
 			(project "block diagram"
-				(path "/290c0625-1e23-4ef7-8910-f1eb5378fd87/46229e74-cb6e-4f48-8e10-26ccf9ffc6c9"
+				(path "/290c0625-1e23-4ef7-8910-f1eb5378fd87/645251e2-b784-4e24-8757-44ff6e2afd31"
 					(reference "R5")
 					(unit 1)
@@
 		(on_board yes)
 		(dnp no)
-		(property "Reference" "#PWR04"
+		(property "Reference" "#PWR02"
 			(at 156.21 27.94 0)
 			(effects
@@
 		(instances
 			(project "block diagram"
-				(path "/290c0625-1e23-4ef7-8910-f1eb5378fd87/46229e74-cb6e-4f48-8e10-26ccf9ffc6c9"
-					(reference "#PWR04")
+				(path "/290c0625-1e23-4ef7-8910-f1eb5378fd87/645251e2-b784-4e24-8757-44ff6e2afd31"
+					(reference "#PWR02")
 					(unit 1)
 				)
@@
 		(on_board yes)
 		(dnp no)
-		(property "Reference" "#PWR02"
+		(property "Reference" "#PWR03"
 			(at 185.42 116.84 0)
 			(effects
@@
 		(instances
 			(project "block diagram"
-				(path "/290c0625-1e23-4ef7-8910-f1eb5378fd87/46229e74-cb6e-4f48-8e10-26ccf9ffc6c9"
-					(reference "#PWR02")
+				(path "/290c0625-1e23-4ef7-8910-f1eb5378fd87/645251e2-b784-4e24-8757-44ff6e2afd31"
+					(reference "#PWR03")
 					(unit 1)
 				)
@@
 		(on_board yes)
 		(dnp no)
-		(property "Reference" "R3"
+		(property "Reference" "R1"
 			(at 152.4 60.96 0)
 			(effects
@@
 		(instances
 			(project "block diagram"
-				(path "/290c0625-1e23-4ef7-8910-f1eb5378fd87/46229e74-cb6e-4f48-8e10-26ccf9ffc6c9"
-					(reference "R3")
+				(path "/290c0625-1e23-4ef7-8910-f1eb5378fd87/645251e2-b784-4e24-8757-44ff6e2afd31"
+					(reference "R1")
 					(unit 1)
 				)
@@
 		(instances
 			(project "block diagram"
-				(path "/290c0625-1e23-4ef7-8910-f1eb5378fd87/46229e74-cb6e-4f48-8e10-26ccf9ffc6c9"
+				(path "/290c0625-1e23-4ef7-8910-f1eb5378fd87/645251e2-b784-4e24-8757-44ff6e2afd31"
 					(reference "BZ1")
 					(unit 1)
@@
 		(dnp no)
 		(fields_autoplaced yes)
-		(property "Reference" "U4"
+		(property "Reference" "U3"
 			(at 99.9333 48.26 0)
 			(effects
@@
 		(instances
 			(project "block diagram"
-				(path "/290c0625-1e23-4ef7-8910-f1eb5378fd87/46229e74-cb6e-4f48-8e10-26ccf9ffc6c9"
-					(reference "U4")
+				(path "/290c0625-1e23-4ef7-8910-f1eb5378fd87/645251e2-b784-4e24-8757-44ff6e2afd31"
+					(reference "U3")
 					(unit 1)
 				)
@@
 		(dnp no)
 		(fields_autoplaced yes)
-		(property "Reference" "#PWR03"
+		(property "Reference" "#PWR04"
 			(at 234.95 91.44 0)
 			(effects
@@
 		(instances
 			(project "block diagram"
-				(path "/290c0625-1e23-4ef7-8910-f1eb5378fd87/46229e74-cb6e-4f48-8e10-26ccf9ffc6c9"
-					(reference "#PWR03")
-					(unit 1)
-				)
+				(path "/290c0625-1e23-4ef7-8910-f1eb5378fd87/645251e2-b784-4e24-8757-44ff6e2afd31"
+					(reference "#PWR04")
+					(unit 1)
+				)
