File: prototype/prototype/sensor_mod.kicad_sch (KiCad schematic)
At the start: 12 parts, among them U7 LM393

Commit message: idk
Parts:
- C1: renamed from C9; footprint (none) -> Photon:C0603
- C9: renamed from C10; footprint (none) -> Photon:C0603
- R11: renamed from R15; footprint (none) -> Photon:R_0603_1608Metric_Pad0.98x0.95mm_HandSolder
- R3: renamed from R11; footprint (none) -> Photon:R_0603_1608Metric_Pad0.98x0.95mm_HandSolder
- R4: renamed from R12; footprint (none) -> Photon:R_0603_1608Metric_Pad0.98x0.95mm_HandSolder
- R6: renamed from R14; footprint (none) -> Photon:R_0603_1608Metric_Pad0.98x0.95mm_HandSolder
- gave numbers to parts that had none: 1
- renumbered R13 to R5, U7 to U2, green_resistor to green_resistor1
Connections:
- net AO: now also U2.2 (-); no longer U2.6 (-)
- net DO: now also U2.1; no longer U2.7
Other:
- note added: "- check ground and vcc connections are corrrect - add resistance and capicitance values - check LED polariy - What is this green thing"
- note removed: "- check ground and vcc connections are corrrect - add resistance and capicitance values - check LED polariy -What is this green thing"
- moved on the sheet: C1

Commit message: final schematic organized
Parts:
- removed D1: IRL81A, LED_THT:LED_SideEmitter_Rectangular_W4.5mm_H1.6mm, symbol LED:IRL81A
- removed D2: LED, symbol Device:LED
- removed R5: R_Variable, symbol Device:R_Variable
- removed U2: LM393, symbol Comparator:LM393
- removed U3: MQ-6, Sensor:MQ-6, symbol Sensor_Gas:MQ-6
- removed green_resistor1: R, symbol Device:R
- added BZ1: Buzzer, symbol Device:Buzzer
- added C13, C19, C33, C36: 0.1uF, Photon:C0603, symbol Device:C
- added C14: 10nF, Photon:C0603, symbol Device:C
- added C15: 220uF, Photon:C0603, symbol Device:C
- added C16, C18: 10uF, Photon:C0603, symbol Device:C
- added C17, C31, C32: 22uF, Photon:C0603, symbol Device:C
- added C20, C34: 1uF, Photon:C0603, symbol Device:C
- added D1: 1N4148, Diode_THT:D_DO-35_SOD27_P7.62mm_Horizontal, symbol Diode:1N4148
- added D3_Green2, D3_Green4, D3_Red2, D3_Red4: LED, symbol Device:LED
- added F2: 0.5A, Photon:Fuse_1206_3216Metric, symbol Device:Fuse
- added J2: Conn_01x06_Pin, symbol Connector:Conn_01x06_Pin
- added L2: 10mH, Photon:L_APV_ANR5040, symbol Device:L_Coupled
- added PS2: HLK-5M05, Converter_ACDC:Converter_ACDC_Hi-Link_HLK-5Mxx, symbol Converter_ACDC:HLK-5M05
- added Q5: AO3400, symbol Simulation_SPICE:NMOS
- added Q6, Q7, Q8: 2N7002, symbol Simulation_SPICE:NMOS
- added R12, R13, R14, R15, R22: 4.7k, Photon:R_0603_1608Metric_Pad0.98x0.95mm_HandSolder, symbol Device:R
- added R21, R37, R38: 330, Photon:R_0603_1608Metric_Pad0.98x0.95mm_HandSolder, symbol Device:R
- added R24, R39: 10k, Photon:R_0603_1608Metric_Pad0.98x0.95mm_HandSolder, symbol Device:R
- added R5: 100, Photon:R_0603_1608Metric_Pad0.98x0.95mm_HandSolder, symbol Device:R
- added RV2: 10D561, Photon:RV_Disc_D7mm_W5.7mm_P5mm, symbol Device:Varistor
- added U14, U6: ESP32-WROOM-32E, RF_Module:ESP32-WROOM-32D, symbol RF_Module:ESP32-WROOM-32E
- added U2: MQ-5, Sensor:MQ-6, symbol Sensor_Gas:MQ-6
- added U3: CI121S021 [adc], Package_TO_SOT_SMD:SOT-23-6, symbol Analog_ADC:ADS1110
- added U4: AMS1117-3.3, Package_TO_SOT_SMD:SOT-223-3_TabPin2, symbol Regulator_Linear:AMS1117-3.3
- C1: value C -> 10uF
- C9: value C -> 1uF
- R11: value R -> 330
- R3: value R -> 20k; footprint Photon:R_0603_1608Metric_Pad0.98x0.95mm_HandSolder -> (none)
- R4: value R -> 10k
- R6: value R -> 4.7k
Connections:
- net VCC is gone; now on net +5V: C9.1
- net GND: now also R3.2, R4.2, C14.2, C15.2, C16.2, C17.2, C18.2, C19.2, C20.2, C31.2, C32.2, C33.2, C34.2, C36.2, D3_Green2.1 (K), D3_Green4.1 (K), D3_Red2.1 (K), D3_Red4.1 (K), J2.6 (Pin_6), PS2.3 (-Vout), Q5.3 (S), U14.1 (GND), U14.15 (GND), U14.38 (GND), U14.39 (GND), U2.5 (VH-), U3.2 (GND), U4.1 (GND), U6.1 (GND), U6.15 (GND), U6.38 (GND), U6.39 (GND); no longer R11.2, R3.1, R6.1
- net at R4.1: now also Q5.2 (G), R5.1
- net at R11.1: now also U6.27 (IO16)
- net AO renamed +5V
- net +5V: now also R6.1, BZ1.1 (+), C14.1, C15.1, C16.1, D1.1 (K), PS2.4 (+Vout), R13.1, R14.1, U2.2 (VH+), U2.4 (A2), U2.6 (A1), U3.1 (VA), U4.3 (VI); no longer R6.2
- new net: L2.2, PS2.1 (AC/L)
- new net: L2.4, PS2.2 (AC/N)
- new net: C13.1, F2.2, L2.1, RV2.1
- new net: C13.2, L2.3, RV2.2
- new net: R37.1, U14.27 (IO16)
- new net: D3_Red4.2 (A), R37.2
- new net: D3_Green4.2 (A), R38.2
- new net: BZ1.2 (-), D1.2 (A), Q5.1 (D)
- new net: D3_Green2.2 (A), R21.2
- new net: D3_Red2.2 (A), R11.2
- new net +3.3V: C17.1, C18.1, C19.1, C31.1, C32.1, C33.1, C36.1, J2.1 (Pin_1), Q6.2 (G), Q7.2 (G), Q8.2 (G), R12.1, R15.1, R22.1, R24.1, R39.1, U14.2 (VDD), U4.2 (VO), U6.2 (VDD)
- new net BUZZ_OUT: R5.2
- new net CLK_3: Q8.3 (S), R22.2, U14.30 (IO18), U6.30 (IO18)
- new net CLK_5: Q8.1 (D), R14.2, U3.4 (SCLK)
- new net CS_3: Q6.3 (S), R12.2, U14.14 (IO12), U6.14 (IO12)
- new net CS_5: Q6.1 (D), R6.2, U3.6 (~{CS})
- new net ESP_EN: C20.1, C34.1, J2.2 (Pin_2), R21.1, R24.2, R38.1, R39.2, U14.3 (EN), U6.3 (EN)
- new net ESP_IO0: J2.3 (Pin_3), U14.25 (IO0), U6.25 (IO0)
- new net ESP_RDD0: J2.5 (Pin_5)
- new net ESP_RXD0: U14.34 (RXD0/IO3), U6.34 (RXD0/IO3)
- new net ESP_TXD0: J2.4 (Pin_4), U14.35 (TXD0/IO1), U6.35 (TXD0/IO1)
- new net SDATA_3: Q7.3 (S), R15.2, U14.28 (IO17), U6.28 (IO17)
- new net SDATA_5: Q7.1 (D), R13.2, U3.5 (SDATA)
- new net Sensor_A_O: R3.1, U2.1 (B1), U2.3 (B2), U3.3 (VIN)
Other:
- note added: "Analog to Digital Converter"
- note added: "Buzzer"
- note added: "ESP Program Pins"
- note added: "LDO 5v -> 3.3v"
- note added: "Logic Shifting Circuits"
- note added: "Power Transformer"
- note added: "Sensor Module"
- note removed: "- check ground and vcc connections are corrrect - add resistance and capicitance values - check LED polariy - What is this green thing"
