File: prototype/prototype/block diagram.kicad_pcb (KiCad board)
At the start: 2 copper layers, 80 x 80.5 mm, 39 parts, among them J1 Conn_01x06_Pin, J2 Screw_Terminal_01x02, Q1 2N7002, Q2 2N7002, Q3 2N7002, Q4 AO3400, U1 MQ-5, U11 ESP32-WROOM-32E, U2 CI121S021 [adc], U3 AMS1117-3.3

Commit message: final final pcb ever fr ong
Parts:
- added REF**: MountingHole_3.2mm_M3_ISO7380, MountingHole:MountingHole_3.2mm_M3_ISO7380, F.Cu at (188.4, 55.0)
- added REF**: MountingHole_3.2mm_M3_ISO7380, MountingHole:MountingHole_3.2mm_M3_ISO7380, F.Cu at (113.7, 55.2)
- added REF**: MountingHole_3.2mm_M3_ISO7380, MountingHole:MountingHole_3.2mm_M3_ISO7380, F.Cu at (113.7, 130.2)
Routing:
- net GND: vias 36 -> 48
Other:
- board size 80 x 80.5 mm -> 82.3 x 82.8 mm
- board text added: "ʚɞ"
