File: prototype/prototype/block diagram.kicad_sch (KiCad schematic)
At the start: 40 parts, among them J1 Conn_01x06_Pin, J2 Screw_Terminal_01x02, Q1 2N7002, Q2 AO3400, Q3 2N7002, Q4 2N7002, U1 AMS1117-3.3, U11 ESP32-WROOM-32E, U5 MQ-5, U8 CI121S021 [adc]

Commit message: finished pcb prototype
Connections:
- net ESP_RDD0 is gone; now on net ESP_IO0: J1.5 (Pin_5)
- net CLK_3: now also U11.28 (IO17); no longer U11.30 (IO18)
- net ESP_IO0: no longer J1.3 (Pin_3)
- net ESP_RXD0: now also J1.4 (Pin_4)
- net ESP_TXD0: now also J1.3 (Pin_3); no longer J1.4 (Pin_4)
- net IO_16_on: now also U11.9 (IO33); no longer U11.27 (IO16)
- net SDATA_3: now also U11.30 (IO18); no longer U11.28 (IO17)
Changed lines of the file:
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@@
 	)
 	(label "SDATA_3"
-		(at 132.08 62.23 180)
+		(at 132.08 64.77 180)
 		(effects
 			(font
@@
 	)
 	(label "CLK_3"
-		(at 132.08 64.77 180)
+		(at 132.08 62.23 180)
 		(effects
 			(font
@@
 		)
 	)
-	(label "ESP_RDD0"
-		(at 215.9 95.25 0)
-		(effects
-			(font
-				(size 1.27 1.27)
-			)
-			(justify left bottom)
-		)
-	)
 	(label "CS_5"
 		(at 77.47 137.16 0)
@@
 	)
 	(label "ESP_IO0"
-		(at 215.9 90.17 0)
+		(at 215.9 95.25 0)
 		(effects
 			(font
@@
 	)
 	(label "IO_16_on"
-		(at 132.08 59.69 180)
+		(at 133.35 87.63 180)
 		(effects
 			(font
@@
 	)
 	(label "ESP_TXD0"
+		(at 215.9 90.17 0)
+		(effects
+			(font
+				(size 1.27 1.27)
+			)
+			(justify left bottom)
+		)
+	)
+	(label "ESP_RXD0"
 		(at 215.9 92.71 0)
 		(effects

Commit message: FINAL FINAL PCB
Parts:
- renumbered BZ2 to BZ1, C5 to C1, C12 to C10, C11 to C2, C2 to C3, C3 to C4, C4 to C5, C10 to C9, D3_Red1 to D2, Q4 to Q1, Q3 to Q2, Q1 to Q3, R23 to R1, R9 to R10, R20 to R11, R3 to R12, R19 to R13, R17 to R2, R16 to R3, R7 to R4, R8 to R5, R1 to R6, R2 to R7, R10 to R8, R4 to R9
Changed lines of the file:
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@@
 		(on_board yes)
 		(dnp no)
-		(property "Reference" "R16"
+		(property "Reference" "R3"
 			(at 264.668 152.146 0)
 			(effects
@@
 			(project "block diagram"
 				(path "/290c0625-1e23-4ef7-8910-f1eb5378fd87"
-					(reference "R16")
+					(reference "R3")
 					(unit 1)
 				)
@@
 		(on_board yes)
 		(dnp no)
-		(property "Reference" "R1"
+		(property "Reference" "R6"
 			(at 195.58 138.4299 0)
 			(effects
@@
 			(project "block diagram"
 				(path "/290c0625-1e23-4ef7-8910-f1eb5378fd87"
-					(reference "R1")
+					(reference "R6")
 					(unit 1)
 				)
@@
 		(on_board yes)
 		(dnp no)
-		(property "Reference" "R4"
+		(property "Reference" "R9"
 			(at 124.46 153.67 90)
 			(effects
@@
 			(project ""
 				(path "/290c0625-1e23-4ef7-8910-f1eb5378fd87"
-					(reference "R4")
+					(reference "R9")
 					(unit 1)
 				)
@@
 		(on_board yes)
 		(dnp no)
-		(property "Reference" "Q4"
+		(property "Reference" "Q1"
 			(at 255.27 161.29 90)
 			(effects
@@
 			(project "block diagram"
 				(path "/290c0625-1e23-4ef7-8910-f1eb5378fd87"
-					(reference "Q4")
+					(reference "Q1")
 					(unit 1)
 				)
@@
 		(on_board yes)
 		(dnp no)
-		(property "Reference" "R2"
+		(property "Reference" "R7"
 			(at 212.598 140.716 0)
 			(effects
@@
 			(project "block diagram"
 				(path "/290c0625-1e23-4ef7-8910-f1eb5378fd87"
-					(reference "R2")
+					(reference "R7")
 					(unit 1)
 				)
@@
 		(on_board yes)
 		(dnp no)
-		(property "Reference" "R9"
+		(property "Reference" "R10"
 			(at 267.97 90.424 90)
 			(effects
@@
 			(project "block diagram"
 				(path "/290c0625-1e23-4ef7-8910-f1eb5378fd87"
-					(reference "R9")
+					(reference "R10")
 					(unit 1)
 				)
@@
 		(on_board yes)
 		(dnp no)
-		(property "Reference" "C5"
+		(property "Reference" "C1"
 			(at 67.31 32.512 0)
 			(effects
@@
 			(project "block diagram"
 				(path "/290c0625-1e23-4ef7-8910-f1eb5378fd87"
-					(reference "C5")
+					(reference "C1")
 					(unit 1)
 				)
@@
 		(on_board yes)
 		(dnp no)
-		(property "Reference" "D3_Red1"
+		(property "Reference" "D2"
 			(at 250.952 46.228 0)
 			(effects
@@
 			(project "block diagram"
 				(path "/290c0625-1e23-4ef7-8910-f1eb5378fd87"
-					(reference "D3_Red1")
+					(reference "D2")
 					(unit 1)
 				)
@@
 		(dnp no)
 		(fields_autoplaced yes)
-		(property "Reference" "R7"
+		(property "Reference" "R4"
 			(at 247.65 130.8099 0)
 			(effects
@@
 			(project "block diagram"
 				(path "/290c0625-1e23-4ef7-8910-f1eb5378fd87"
-					(reference "R7")
+					(reference "R4")
 					(unit 1)
 				)
@@
 		(dnp no)
 		(fields_autoplaced yes)
-		(property "Reference" "R23"
+		(property "Reference" "R1"
 			(at 72.39 93.9799 0)
 			(effects
@@
 			(project "block diagram"
 				(path "/290c0625-1e23-4ef7-8910-f1eb5378fd87"
-					(reference "R23")
+					(reference "R1")
 					(unit 1)
 				)
@@
 		(on_board yes)
 		(dnp no)
-		(property "Reference" "Q3"
+		(property "Reference" "Q2"
 			(at 254 142.24 90)
 			(effects
@@
 			(project "block diagram"
 				(path "/290c0625-1e23-4ef7-8910-f1eb5378fd87"
-					(reference "Q3")
+					(reference "Q2")
 					(unit 1)
 				)
@@
 		(on_board yes)
 		(dnp no)
-		(property "Reference" "C3"
+		(property "Reference" "C4"
 			(at 41.91 137.1599 0)
 			(effects
@@
 			(project "block diagram"
 				(path "/290c0625-1e23-4ef7-8910-f1eb5378fd87"
-					(reference "C3")
+					(reference "C4")
 					(unit 1)
 				)
@@
 		(dnp no)
 		(fields_autoplaced yes)
-		(property "Reference" "R20"
+		(property "Reference" "R11"
 			(at 264.16 97.7899 0)
 			(effects
@@
 			(project "block diagram"
 				(path "/290c0625-1e23-4ef7-8910-f1eb5378fd87"
-					(reference "R20")
+					(reference "R11")
 					(unit 1)
 				)
@@
 		(dnp no)
 		(fields_autoplaced yes)
-		(property "Reference" "C12"
+		(property "Reference" "C10"
 			(at 71.12 179.0699 0)
 			(effects
@@
 			(project "block diagram"
 				(path "/290c0625-1e23-4ef7-8910-f1eb5378fd87"
-					(reference "C12")
+					(reference "C10")
 					(unit 1)
 				)
@@
 		(on_board yes)
 		(dnp no)
-		(property "Reference" "Q1"
+		(property "Reference" "Q3"
 			(at 203.2 149.86 90)
 			(effects
@@
 			(project "block diagram"
 				(path "/290c0625-1e23-4ef7-8910-f1eb5378fd87"
-					(reference "Q1")
+					(reference "Q3")
 					(unit 1)
 				)
@@
 		(dnp no)
 		(fields_autoplaced yes)
-		(property "Reference" "R10"
+		(property "Reference" "R8"
 			(at 214.63 45.72 90)
 			(effects
@@
 			(project "block diagram"
 				(path "/290c0625-1e23-4ef7-8910-f1eb5378fd87"
-					(reference "R10")
+					(reference "R8")
 					(unit 1)
 				)
@@
 		(on_board yes)
 		(dnp no)
-		(property "Reference" "R17"
+		(property "Reference" "R2"
 			(at 247.65 149.8599 0)
 			(effects
@@
 			(project "block diagram"
 				(path "/290c0625-1e23-4ef7-8910-f1eb5378fd87"
-					(reference "R17")
+					(reference "R2")
 					(unit 1)
 				)
@@
 		(on_board yes)
 		(dnp no)
-		(property "Reference" "R8"
+		(property "Reference" "R5"
 			(at 267.97 132.0799 0)
 			(effects
@@
 			(project "block diagram"
 				(path "/290c0625-1e23-4ef7-8910-f1eb5378fd87"
-					(reference "R8")
+					(reference "R5")
 					(unit 1)
 				)
@@
 		(dnp no)
 		(fields_autoplaced yes)
-		(property "Reference" "C4"
+		(property "Reference" "C5"
 			(at 153.67 149.8599 0)
 			(effects
@@
 			(project "block diagram"
 				(path "/290c0625-1e23-4ef7-8910-f1eb5378fd87"
-					(reference "C4")
+					(reference "C5")
 					(unit 1)
 				)
@@
 		(dnp no)
 		(fields_autoplaced yes)
-		(property "Reference" "R3"
+		(property "Reference" "R12"
 			(at 259.08 82.5499 0)
 			(effects
@@
 			(project "block diagram"
 				(path "/290c0625-1e23-4ef7-8910-f1eb5378fd87"
-					(reference "R3")
+					(reference "R12")
 					(unit 1)
 				)
@@
 		(on_board yes)
 		(dnp no)
-		(property "Reference" "BZ2"
+		(property "Reference" "BZ1"
 			(at 246.38 82.5499 0)
 			(effects
@@
 			(project "block diagram"
 				(path "/290c0625-1e23-4ef7-8910-f1eb5378fd87"
-					(reference "BZ2")
+					(reference "BZ1")
 					(unit 1)
 				)
@@
 		(dnp no)
 		(fields_autoplaced yes)
-		(property "Reference" "R19"
+		(property "Reference" "R13"
 			(at 260.35 45.72 90)
 			(effects
@@
 			(project "block diagram"
 				(path "/290c0625-1e23-4ef7-8910-f1eb5378fd87"
-					(reference "R19")
+					(reference "R13")
 					(unit 1)
 				)
@@
 		(on_board yes)
 		(dnp no)
-		(property "Reference" "C10"
+		(property "Reference" "C9"
 			(at 34.29 179.07 0)
 			(effects
@@
 			(project "block diagram"
 				(path "/290c0625-1e23-4ef7-8910-f1eb5378fd87"
-					(reference "C10")
+					(reference "C9")
 					(unit 1)
 				)
@@
 		(dnp no)
 		(fields_autoplaced yes)
-		(property "Reference" "C2"
+		(property "Reference" "C3"
 			(at 52.07 137.1599 0)
 			(effects
@@
 			(project "block diagram"
 				(path "/290c0625-1e23-4ef7-8910-f1eb5378fd87"
-					(reference "C2")
+					(reference "C3")
 					(unit 1)
 				)
@@
 		(on_board yes)
 		(dnp no)
-		(property "Reference" "C11"
+		(property "Reference" "C2"
 			(at 27.432 84.836 0)
 			(effects
@@
 			(project "block diagram"
 				(path "/290c0625-1e23-4ef7-8910-f1eb5378fd87"
-					(reference "C11")
+					(reference "C2")
 					(unit 1)
 				)

Commit message: final final pcb ever fr ong
Parts:
- J3: renamed from J1; footprint Connector_Hirose:Hirose_DF13-06P-1.25DS_1x06_P1.25mm_Horizontal -> Connector_JST:JST_EH_S6B-EH_1x06_P2.50mm_Horizontal
- renumbered TP3 to 3V2, TP1 to 5V2, BZ1 to BZ2, C7 to C10, C6 to C11, C4 to C3, C9 to C4, C3 to C5, C1 to C6, C10 to C7, C5 to C8, C8 to C9, D1 to D2, D2 to D3, PS1 to PS2, Q3 to Q2, Q2 to Q3, Q2 to Q4, Q1 to Q5, R13 to R10, R5 to R12, R3 to R13, R10 to R14, R1 to R2, R9 to R3, R6 to R4, R8 to R5, R7 to R6, R4 to R7, R2 to R8, R12 to R9, U5 to U2, U1 to U3, U8 to U4, U11 to U5
